File: nodes/hardware/SenseMate/SenseMatePCB/SenseMatePCB.kicad_sch (KiCad schematic)
At the start: 13 parts, among them J1 Conn_01x04, M1 Motor_DC, Q1 2SC1815, Q2 2SC1815, SW5 SW_DPDT_x2

Commit message: changed motor connector to 2-pin-header
Parts:
- M1: footprint Connector_JST:JST_PH_S2B-PH-K_1x02_P2.00mm_Horizontal -> Connector_PinHeader_2.54mm:PinHeader_1x02_P2.54mm_Vertical
Changed lines of the file:
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@@
 			)
 		)
-		(property "Footprint" "Connector_JST:JST_PH_S2B-PH-K_1x02_P2.00mm_Horizontal"
+		(property "Footprint" "Connector_PinHeader_2.54mm:PinHeader_1x02_P2.54mm_Vertical"
 			(at 147.32 155.194 0)
 			(effects
